Commit message: Added Gazebo world, ros2_control, and robot updates

File: description/robo_core.xacro (robot description, xacro)
@@ -70,4 +70,11 @@
     </xacro:inertial_box>
   </link>
+  <gazebo reference="chassis">
+    <material>Gazebo/White</material>
+    <mu1>1.0</mu1>
+    <mu2>1.0</mu2>
+    <kp>1000000.0</kp>
+    <kd>100.0</kd>
+  </gazebo>
   <!-- ═══════════ LEFT DRIVE WHEEL ═══════════ -->
   <!--
@@ -105,4 +112,12 @@
     </xacro:inertial_cylinder>
   </link>
+  <gazebo reference="left_wheel">
+    <material>Gazebo/Blue</material>
+    <mu1>10.0</mu1>
+    <mu2>10.0</mu2>
+    <kp>1000000.0</kp>
+    <kd>100.0</kd>
+    <fdir1>1 0 0</fdir1>
+  </gazebo>
   <!-- ═══════════ RIGHT DRIVE WHEEL ═══════════ -->
   <!--
@@ -131,8 +146,16 @@
       </geometry>
     </collision>
-    <xacro:inertial_cylinder mass="0.2" length="0.04" radius="0.0565">
+    <xacro:inertial_cylinder mass="0.1" length="0.04" radius="0.0565">
       <origin xyz="0 0 0" rpy="0 0 0"/>
     </xacro:inertial_cylinder>
   </link>
+  <gazebo reference="right_wheel">
+    <material>Gazebo/Blue</material>
+    <mu1>10.0</mu1>
+    <mu2>10.0</mu2>
+    <kp>1000000.0</kp>
+    <kd>100.0</kd>
+    <fdir1>1 0 0</fdir1>
+  </gazebo>
   <!-- ═══════════ CASTER WHEELS (4 CORNERS) ═══════════ -->
   <!-- x = ±0.18 (half-length 0.23 − 5cm inset)
@@ -151,4 +174,9 @@
     </xacro:inertial_sphere>
   </link>
+  <gazebo reference="caster_front_left">
+    <material>Gazebo/Black</material>
+    <mu1>0.001</mu1>
+    <mu2>0.001</mu2>
+  </gazebo>
   <joint name="caster_front_right_joint" type="fixed">
     <parent link="chassis"/>
@@ -163,4 +191,9 @@
     </xacro:inertial_sphere>
   </link>
+  <gazebo reference="caster_front_right">
+    <material>Gazebo/Black</material>
+    <mu1>0.001</mu1>
+    <mu2>0.001</mu2>
+  </gazebo>
   <joint name="caster_rear_left_joint" type="fixed">
     <parent link="chassis"/>
@@ -175,4 +208,9 @@
     </xacro:inertial_sphere>
   </link>
+  <gazebo reference="caster_rear_left">
+    <material>Gazebo/Black</material>
+    <mu1>0.001</mu1>
+    <mu2>0.001</mu2>
+  </gazebo>
   <joint name="caster_rear_right_joint" type="fixed">
     <parent link="chassis"/>
@@ -187,3 +225,8 @@
     </xacro:inertial_sphere>
   </link>
+  <gazebo reference="caster_rear_right">
+    <material>Gazebo/Black</material>
+    <mu1>0.001</mu1>
+    <mu2>0.001</mu2>
+  </gazebo>
 </robot>

File: description/robot.urdf.xacro (robot description, xacro)
@@ -2,3 +2,5 @@
 <robot xmlns:xacro="http://www.ros.org/wiki/xacro"  name="robot">
     <xacro:include filename="robo_core.xacro" />
+    <xacro:include filename="gazebo_control.xacro" />
+    <xacro:include filename="lidar.xacro" />
 </robot>
